File: CAO/KiCAD/Detecteur_de_train/Detecteur_de_train.kicad_sch (KiCad schematic)
At the start: 43 parts, among them J1 Alimentation, J2 Sortie, U1 LMV358IDR, U2 LMV331, U3 MCP6541

Commit message: Update Detecteur_de_train.kicad_sch
Parts:
- added C13, C14: 1u, symbol Device:C
- added TP10: VEE, symbol Connector:TestPoint
- added U5: ~, symbol MesSymboles:MAX1719EUT+T
Connections:
- net GND: now also C14.1, U5.4 (GD), U5.5 (SHDN)
- net VCC: now also U5.2 (IN)
- net VEE: now also C14.2, TP10.1, U5.1 (OUT)
- new net: C13.2, U5.3 (C1-)
- new net: C13.1, U5.6 (C1+)
Other:
- note added: "* Convertisseur DC-DC * Pompe de charge inverseuse * Vin = 5v => Vout = -5V"
- moved on the sheet: C1, C10, C2, C3, C9, D4, J1, R10, R11, R12, R14, R15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

Commit message: Update Detecteur_de_train.kicad_sch
Parts:
- renumbered C8 to C11, C9 to C12, C4 to C2, C2 to C3, C3 to C4, C13 to C7, C14 to C8, C7 to C9, R11 to R10, R8 to R11, R9 to R12, R14 to R13, R15 to R14, R12 to R8, R10 to R9, TP7 to TP2, TP2 to TP3, TP3 to TP4, TP10 to TP5, TP4 to TP6, TP5 to TP7, TP6 to TP8, TP8 to TP9, U5 to U2, U2 to U3, U3 to U4

Commit message: Update Detecteur_de_train.kicad_sch
Parts:
- added H1, H2: MountingHole, symbol Mechanical:MountingHole
Changed lines of the file:
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@@
+    )
+  )
+  (symbol (lib_id "Mechanical:MountingHole") (at 26.67 189.23 0) (unit 1)
+    (in_bom yes) (on_board yes) (dnp no)
+    (property "Reference" "H2" (at 25.4 182.88 0)
+      (effects (font (size 1.27 1.27)) (justify left))
+    )
+    (property "Value" "MountingHole" (at 21.59 185.42 0)
+      (effects (font (size 1.27 1.27)) (justify left))
+    )
+    (property "Footprint" "" (at 26.67 189.23 0)
+      (effects (font (size 1.27 1.27)) hide)
+    )
+    (property "Datasheet" "~" (at 26.67 189.23 0)
+      (effects (font (size 1.27 1.27)) hide)
+    )
+    (instances
+      (project "Detecteur_de_train"
+        (path "/d1ba9e77-4071-4db6-81fc-bb548139ea63"
+          (reference "H2") (unit 1)
+        )
+      )
     )
   )
@@
     )
   )
+  (symbol (lib_id "Mechanical:MountingHole") (at 26.67 176.53 0) (unit 1)
+    (in_bom yes) (on_board yes) (dnp no)
+    (property "Reference" "H1" (at 25.4 171.45 0)
+      (effects (font (size 1.27 1.27)) (justify left))
+    )
+    (property "Value" "MountingHole" (at 21.59 173.99 0)
+      (effects (font (size 1.27 1.27)) (justify left))
+    )
+    (property "Footprint" "" (at 26.67 176.53 0)
+      (effects (font (size 1.27 1.27)) hide)
+    )
+    (property "Datasheet" "~" (at 26.67 176.53 0)
+      (effects (font (size 1.27 1.27)) hide)
+    )
+    (instances
+      (project "Detecteur_de_train"
+        (path "/d1ba9e77-4071-4db6-81fc-bb548139ea63"
+          (reference "H1") (unit 1)
+        )
+      )
+    )
+  )
   (symbol (lib_id "power:GND") (at 107.95 144.78 0) (unit 1)
     (in_bom yes) (on_board yes) (dnp no)
@@
     )
   )
-  (symbol (lib_id "Device:C") (at 93.98 130.81 90) (unit 1)
-    (in_bom yes) (on_board yes) (dnp no)
-    (property "Reference" "C5" (at 91.44 128.27 90)
-      (effects (font (size 1.27 1.27)))
-    )
-    (property "Value" "10n" (at 96.52 128.27 90)
-      (effects (font (size 1.27 1.27)))
-    )
-    (property "Footprint" "" (at 97.79 129.8448 0)
+  (symbol (lib_name "C_1") (lib_id "Device:C") (at 93.98 130.81 90) (unit 1)
+    (in_bom yes) (on_board yes) (dnp no)
+    (property "Reference" "C5" (at 96.52 133.35 90)
+      (effects (font (size 1.27 1.27)))
+    )
+    (property "Value" "10n" (at 91.44 133.35 90)
+      (effects (font (size 1.27 1.27)))
+    )
+    (property "Footprint" "" (at 90.17 131.7752 0)
       (effects (font (size 1.27 1.27)) hide)
     )
@@
     )
   )
-  (symbol (lib_id "Device:C") (at 52.07 149.86 90) (unit 1)
-    (in_bom yes) (on_board yes) (dnp no)
-    (property "Reference" "C2" (at 48.26 147.32 90)
-      (effects (font (size 1.27 1.27)))
-    )
-    (property "Value" "10p" (at 55.88 147.32 90)
-      (effects (font (size 1.27 1.27)))
-    )
-    (property "Footprint" "" (at 55.88 148.8948 0)
-      (effects (font (size 1.27 1.27)) hide)
-    )
+  (symbol (lib_name "C_2") (lib_id "Device:C") (at 52.07 149.86 90) (unit 1)
+    (in_bom yes) (on_board yes) (dnp no)
+    (property "Reference" "C2" (at 49.53 153.67 90)
+      (effects (font (size 1.27 1.27)))
+    )
+    (property "Value" "10p" (at 49.53 146.05 90)
+      (effects (font (size 1.27 1.27)))
+    )
+    (property "Footprint" "" (at 51.1048 146.05 0)
+      (effects (font (size 1.27 1.27)) hide)
+    )

Commit message: Update Detecteur_de_train.kicad_sch
Parts:
- C1: footprint (none) -> Capacitor_SMD:CP_Elec_5x5.4
- C10, C11, C12, C2, C3, C4, C5, C6, C7, C8, C9: footprint (none) -> Capacitor_SMD:C_0805_2012Metric_Pad1.18x1.45mm_HandSolder
- D1: footprint LED_THT:LED_D5.0mm_IRGrey -> Connector_PinSocket_2.54mm:PinSocket_1x02_P2.54mm_Vertical
- D3: footprint (none) -> LED_SMD:LED_0805_2012Metric_Pad1.15x1.40mm_HandSolder
- D4: footprint (none) -> Connector_PinSocket_2.54mm:PinSocket_1x02_P2.54mm_Vertical
- H1, H2: footprint (none) -> MountingHole:MountingHole_3mm_Pad
- J1: footprint (none) -> Connector_PinHeader_2.54mm:PinHeader_1x03_P2.54mm_Vertical
- R1, R10, R11, R12, R13, R14, R2, R3, R4, R5, R6, R7, R8, R9: footprint (none) -> Resistor_SMD:R_0805_2012Metric_Pad1.20x1.40mm_HandSolder
- U4: footprint Package_TO_SOT_SMD:SOT-23-5 -> Package_TO_SOT_SMD:SOT-23-6_Handsoldering
Changed lines of the file:
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@@
       (effects (font (size 1.27 1.27)) (justify left))
     )
-    (property "Footprint" "" (at 26.67 189.23 0)
+    (property "Footprint" "MountingHole:MountingHole_3mm_Pad" (at 26.67 189.23 0)
       (effects (font (size 1.27 1.27)) hide)
     )
@@
       (effects (font (size 1.27 1.27)) (justify left))
     )
-    (property "Footprint" "" (at 258.826 68.834 90)
+    (property "Footprint" "Resistor_SMD:R_0805_2012Metric_Pad1.20x1.40mm_HandSolder" (at 258.826 68.834 90)
       (effects (font (size 1.27 1.27)) hide)
     )
@@
       (effects (font (size 1.27 1.27)))
     )
-    (property "Footprint" "" (at 234.95 37.1348 0)
+    (property "Footprint" "Capacitor_SMD:C_0805_2012Metric_Pad1.18x1.45mm_HandSolder" (at 234.95 37.1348 0)
       (effects (font (size 1.27 1.27)) hide)
     )
@@
       (effects (font (size 1.27 1.27)) (justify right))
     )
-    (property "Footprint" "" (at 203.5048 83.82 0)
+    (property "Footprint" "Capacitor_SMD:C_0805_2012Metric_Pad1.18x1.45mm_HandSolder" (at 203.5048 83.82 0)
       (effects (font (size 1.27 1.27)) hide)
     )
@@
       (effects (font (size 1.27 1.27)))
     )
-    (property "Footprint" "" (at 213.614 47.244 90)
+    (property "Footprint" "Resistor_SMD:R_0805_2012Metric_Pad1.20x1.40mm_HandSolder" (at 213.614 47.244 90)
       (effects (font (size 1.27 1.27)) hide)
     )
@@
       (effects (font (size 1.27 1.27)))
     )
-    (property "Footprint" "" (at 192.786 125.984 90)
+    (property "Footprint" "Resistor_SMD:R_0805_2012Metric_Pad1.20x1.40mm_HandSolder" (at 192.786 125.984 90)
       (effects (font (size 1.27 1.27)) hide)
     )
@@
       (effects (font (size 1.27 1.27)) (justify right))
     )
-    (property "Footprint" "" (at 231.14 151.13 0)
+    (property "Footprint" "LED_SMD:LED_0805_2012Metric_Pad1.15x1.40mm_HandSolder" (at 231.14 151.13 0)
       (effects (font (size 1.27 1.27)) hide)
     )
@@
       (effects (font (size 1.27 1.27)) (justify left))
     )
-    (property "Footprint" "" (at 44.45 46.99 0)
+    (property "Footprint" "Capacitor_SMD:CP_Elec_5x5.4" (at 44.45 46.99 0)
       (effects (font (size 1.27 1.27)) hide)
     )
@@
       (effects (font (size 1.27 1.27)))
     )
-    (property "Footprint" "" (at 52.324 141.224 90)
+    (property "Footprint" "Resistor_SMD:R_0805_2012Metric_Pad1.20x1.40mm_HandSolder" (at 52.324 141.224 90)
       (effects (font (size 1.27 1.27)) hide)
     )
@@
       (effects (font (size 1.27 1.27)) (justify left))
     )
-    (property "Footprint" "" (at 206.756 43.434 90)
+    (property "Footprint" "Resistor_SMD:R_0805_2012Metric_Pad1.20x1.40mm_HandSolder" (at 206.756 43.434 90)
       (effects (font (size 1.27 1.27)) hide)
     )
@@
       (effects (font (size 1.27 1.27)) (justify left))
     )
-    (property "Footprint" "" (at 61.9252 50.8 0)
+    (property "Footprint" "Capacitor_SMD:C_0805_2012Metric_Pad1.18x1.45mm_HandSolder" (at 61.9252 50.8 0)
       (effects (font (size 1.27 1.27)) hide)
     )
@@
       (effects (font (size 1.27 1.27)))
     )
-    (property "Footprint" "" (at 106.934 138.176 90)
+    (property "Footprint" "Resistor_SMD:R_0805_2012Metric_Pad1.20x1.40mm_HandSolder" (at 106.934 138.176 90)
       (effects (font (size 1.27 1.27)) hide)
     )
@@
       (effects (font (size 1.27 1.27)) (justify left))
     )
-    (property "Footprint" "" (at 218.44 123.4948 0)
+    (property "Footprint" "Capacitor_SMD:C_0805_2012Metric_Pad1.18x1.45mm_HandSolder" (at 218.44 123.4948 0)
       (effects (font (size 1.27 1.27)) hide)
     )
@@
       (effects (font (size 1.27 1.27)))
     )
-    (property "Footprint" "" (at 198.374 57.404 90)
+    (property "Footprint" "Resistor_SMD:R_0805_2012Metric_Pad1.20x1.40mm_HandSolder" (at 198.374 57.404 90)
       (effects (font (size 1.27 1.27)) hide)
     )
@@
       (effects (font (size 1.27 1.27)) (justify left))
     )
-    (property "Footprint" "" (at 26.67 176.53 0)
+    (property "Footprint" "MountingHole:MountingHole_3mm_Pad" (at 26.67 176.53 0)
       (effects (font (size 1.27 1.27)) hide)
     )
@@
       (effects (font (size 1.27 1.27)))
     )
-    (property "Footprint" "LED_THT:LED_D5.0mm_IRGrey" (at 33.02 145.415 0)
+    (property "Footprint" "Connector_PinSocket_2.54mm:PinSocket_1x02_P2.54mm_Vertical" (at 33.02 145.415 0)
       (effects (font (size 1.27 1.27)) hide)
     )
@@
       (effects (font (size 1.27 1.27)) (justify right))
     )
-    (property "Footprint" "" (at 257.81 80.01 0)
+    (property "Footprint" "Connector_PinSocket_2.54mm:PinSocket_1x02_P2.54mm_Vertical" (at 257.81 80.01 0)
       (effects (font (size 1.27 1.27)) hide)
     )
@@
       (effects (font (size 1.27 1.27)))
     )
-    (property "Footprint" "" (at 135.636 143.256 90)
+    (property "Footprint" "Resistor_SMD:R_0805_2012Metric_Pad1.20x1.40mm_HandSolder" (at 135.636 143.256 90)
       (effects (font (size 1.27 1.27)) hide)
     )
@@
       (effects (font (size 1.27 1.27)))
     )
-    (property "Footprint" "" (at 232.156 129.794 90)
+    (property "Footprint" "Resistor_SMD:R_0805_2012Metric_Pad1.20x1.40mm_HandSolder" (at 232.156 129.794 90)
       (effects (font (size 1.27 1.27)) hide)
     )
@@
       (effects (font (size 1.27 1.27)))
     )
-    (property "Footprint" "" (at 232.156 142.494 90)
+    (property "Footprint" "Resistor_SMD:R_0805_2012Metric_Pad1.20x1.40mm_HandSolder" (at 232.156 142.494 90)
       (effects (font (size 1.27 1.27)) hide)
     )
@@
       (effects (font (size 1.27 1.27)) (justify left))
     )
-    (property "Footprint" "" (at 173.6852 144.78 0)
+    (property "Footprint" "Capacitor_SMD:C_0805_2012Metric_Pad1.18x1.45mm_HandSolder" (at 173.6852 144.78 0)
       (effects (font (size 1.27 1.27)) hide)
     )
@@
       (effects (font (size 1.27 1.27)))
     )
-    (property "Footprint" "" (at 124.714 148.336 90)
+    (property "Footprint" "Resistor_SMD:R_0805_2012Metric_Pad1.20x1.40mm_HandSolder" (at 124.714 148.336 90)
       (effects (font (size 1.27 1.27)) hide)
     )
@@
       (effects (font (size 1.27 1.27)) (justify left))
     )
-    (property "Footprint" "" (at 27.94 54.61 0)
+    (property "Footprint" "Connector_PinHeader_2.54mm:PinHeader_1x03_P2.54mm_Vertical" (at 27.94 54.61 0)
       (effects (font (size 1.27 1.27)) hide)
     )
@@
       (effects (font (size 1.27 1.27)))
     )
-    (property "Footprint" "" (at 90.17 131.7752 0)
+    (property "Footprint" "Capacitor_SMD:C_0805_2012Metric_Pad1.18x1.45mm_HandSolder" (at 90.17 131.7752 0)
       (effects (font (size 1.27 1.27)) hide)
     )
@@
       (effects (font (size 1.27 1.27)) (justify left))
     )
-    (property "Footprint" "" (at 61.9252 63.5 0)
+    (property "Footprint" "Capacitor_SMD:C_0805_2012Metric_Pad1.18x1.45mm_HandSolder" (at 61.9252 63.5 0)
       (effects (font (size 1.27 1.27)) hide)
     )
@@
       (effects (font (size 1.27 1.27)))
     )
-    (property "Footprint" "" (at 164.1348 55.88 0)
+    (property "Footprint" "Capacitor_SMD:C_0805_2012Metric_Pad1.18x1.45mm_HandSolder" (at 164.1348 55.88 0)
       (effects (font (size 1.27 1.27)) hide)
     )
@@
       (effects (font (size 1.27 1.27)))
     )
-    (property "Footprint" "" (at 237.744 78.994 90)
+    (property "Footprint" "Resistor_SMD:R_0805_2012Metric_Pad1.20x1.40mm_HandSolder" (at 237.744 78.994 90)
       (effects (font (size 1.27 1.27)) hide)
     )
@@
       (effects (font (size 1.27 1.27)))
     )
-    (property "Footprint" "" (at 51.1048 146.05 0)
+    (property "Footprint" "Capacitor_SMD:C_0805_2012Metric_Pad1.18x1.45mm_HandSolder" (at 51.1048 146.05 0)
       (effects (font (size 1.27 1.27)) hide)
     )
@@
       (effects (font (size 1.27 1.27)))
     )
-    (property "Footprint" "Package_TO_SOT_SMD:SOT-23-5" (at 226.06 66.04 0)
+    (property "Footprint" "Package_TO_SOT_SMD:SOT-23-6_Handsoldering" (at 226.06 66.04 0)
       (effects (font (size 1.27 1.27)) (justify left) hide)
     )
@@
       (effects (font (size 1.27 1.27)))
     )
-    (property "Footprint" "" (at 97.79 138.7348 0)
+    (property "Footprint" "Capacitor_SMD:C_0805_2012Metric_Pad1.18x1.45mm_HandSolder" (at 97.79 138.7348 0)
       (effects (font (size 1.27 1.27)) hide)
     )
@@
       (effects (font (size 1.27 1.27)))
     )
-    (property "Footprint" "" (at 147.32 46.0248 0)
+    (property "Footprint" "Capacitor_SMD:C_0805_2012Metric_Pad1.18x1.45mm_HandSolder" (at 147.32 46.0248 0)
       (effects (font (size 1.27 1.27)) hide)
     )
@@
       (effects (font (size 1.27 1.27)))
     )
-    (property "Footprint" "" (at 167.386 141.224 90)
+    (property "Footprint" "Resistor_SMD:R_0805_2012Metric_Pad1.20x1.40mm_HandSolder" (at 167.386 141.224 90)
       (effects (font (size 1.27 1.27)) hide)
     )
@@
       (effects (font (size 1.27 1.27)))
     )
-    (property "Footprint" "" (at 192.786 143.764 90)
-      (effects (font (size 1.27 1.27)) hide)
-    )
+    (property "Footprint" "Resistor_SMD:R_0805_2012Metric_Pad1.20x1.40mm_HandSolder" (at 192.786 143.764 90)
+      (effects (font (size 1.27 1.27)) hide)
+    )

Commit message: Update Detecteur_de_train.kicad_sch
Parts:
- J2: footprint (none) -> Connector_PinHeader_2.54mm:PinHeader_1x02_P2.54mm_Vertical
Changed lines of the file:
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@@
       (effects (font (size 1.27 1.27)) (justify left))
     )
-    (property "Footprint" "" (at 251.46 138.43 0)
+    (property "Footprint" "Connector_PinHeader_2.54mm:PinHeader_1x02_P2.54mm_Vertical" (at 251.46 138.43 0)
       (effects (font (size 1.27 1.27)) hide)
     )
